Commit message: added camera sensor

File: my_robot_description/urdf/camera.xacro (robot description, xacro)
@@ -24,3 +24,15 @@
         <origin xyz="${(base_length+camera_length)/2} 0 ${base_height/2}"  rpy="0 0 0"/>
     </joint>
+    <gazebo reference="camera_link">
+        <material>Gazebo/Red</material>
+        <sensor name="camera_sensor" type="camera">
+            <pose>0 0 0 0 0 0</pose>
+            <visualize>true</visualize>
+            <update_rate>10.0</update_rate>
+            <plugin name="plugin_name" filename="libgazebo_ros_camera.so">
+                <!-- Set TF frame name. If empty, defaults to link name -->
+                <frame_name>camera_link</frame_name>
+            </plugin>
+        </sensor>
+    </gazebo>
 </robot>
