Commit message: Added ros plugins

File: my_robot_description/urdf/mobile_base.xacro (robot description, xacro)
@@ -6,5 +6,5 @@
     <xacro:property name="wheel_raidus" value="0.1"/>
     <xacro:property name="wheel_length" value="0.05"/>
-    <link name="base_footprint_link"/>
+    <link name="base_footprint"/>
     <link name="base_link">
         <visual>
@@ -98,5 +98,5 @@
     </joint>
     <joint name="base_base_footprint_joint" type="fixed">
-        <parent link ="base_footprint_link"/>
+        <parent link ="base_footprint"/>
         <child link="base_link"/>
         <origin xyz="0 0 ${wheel_raidus}" rpy="0 0 0"/>

File: my_robot_description/urdf/my_robot.urdf.xacro (robot description, xacro)
@@ -3,3 +3,4 @@
     <xacro:include  filename="common_properties.xacro"/>
     <xacro:include  filename="mobile_base.xacro"/>
+    <xacro:include  filename="mobile_base_gazebo.xacro"/>
 </robot>

Commit message: Shifted to gazebo classic approach

File: my_robot_description/urdf/mobile_base.xacro (robot description, xacro)
@@ -6,5 +6,5 @@
     <xacro:property name="wheel_raidus" value="0.1"/>
     <xacro:property name="wheel_length" value="0.05"/>
-    <link name="base_footprint"/>
+    <link name="base_footprint_link"/>
     <link name="base_link">
         <visual>
@@ -98,5 +98,5 @@
     </joint>
     <joint name="base_base_footprint_joint" type="fixed">
-        <parent link ="base_footprint"/>
+        <parent link ="base_footprint_link"/>
         <child link="base_link"/>
         <origin xyz="0 0 ${wheel_raidus}" rpy="0 0 0"/>

File: my_robot_description/urdf/mobile_base_gazebo.xacro (robot description, xacro)
@@ -1,5 +1,5 @@
 <?xml version="1.0"?>
 <robot xmlns:xacro="http://www.ros.org/wiki/xacro" >
-    <gazebo reference="caster_wheel_link">
+    <!-- <gazebo reference="caster_wheel_link">
         <mul1 value="0.1"/>
         <mul2 value="0.1"/>
@@ -24,4 +24,16 @@
             <joint_name>base_right_wheel_joint</joint_name>
         </plugin>
+    </gazebo> -->
+    <gazebo reference="base_link">
+        <material>Gazebo/Blue</material>
+    </gazebo>
+    <gazebo reference="right_wheel_link">
+        <material>Gazebo/Grey</material>
+    </gazebo>
+    <gazebo reference="left_wheel_link">
+        <material>Gazebo/Grey</material>
+    </gazebo>
+    <gazebo reference="caster_wheel_link">
+        <material>Gazebo/Grey</material>
     </gazebo>
 </robot>

Commit message: Combined the robot arm with the base

File: my_robot_description/urdf/mobile_base.xacro (robot description, xacro)
@@ -102,4 +102,9 @@
         <origin xyz="0 0 ${wheel_raidus}" rpy="0 0 0"/>
     </joint>
+    <joint name="arm_base_base_joint" type="fixed">
+        <parent link ="base_link"/>
+        <child link="arm_base_link"/>
+        <origin xyz="${(base_length-arm_base_length)/2} 0 ${base_height}" rpy="0 0 0"/>
+    </joint>
     <!-- <link name="second_link">
         <visual>
